Commit message: Rebiuld description files, fix some errors.

File: src/mp500lwa4d_description/urdf/arm/arm.gazebo.xacro (robot description, xacro)
@@ -1,43 +1,44 @@
 <?xml version="1.0"?>
 <robot xmlns:xacro="http://www.ros.org/wiki/xacro">
+    <!--<xacro:include filename="$(find mp500lwa4d_description)/urdf/common.xacro" />-->
     <gazebo reference="arm_base_link">
         <gravity>true</gravity>
         <self_collide>false</self_collide>
-        <material value="Schunk/Black"/>
+        <material value="Gazebo/Black"/>
     </gazebo>
     <gazebo reference="arm_1_link">
         <gravity>true</gravity>
         <self_collide>false</self_collide>
-        <material value="Schunk/LightGrey"/>
+        <material value="Gazebo/Grey"/>
     </gazebo>
     <gazebo reference="arm_2_link">
         <gravity>true</gravity>
         <self_collide>false</self_collide>
-        <material value="Schunk/Black"/>
+        <material value="Gazebo/Black"/>
     </gazebo>
     <gazebo reference="arm_3_link">
         <gravity>true</gravity>
         <self_collide>false</self_collide>
-        <material value="Schunk/LightGrey"/>
+        <material value="Gazebo/Grey"/>
     </gazebo>
     <gazebo reference="arm_4_link">
         <gravity>true</gravity>
         <self_collide>false</self_collide>
-        <material value="Schunk/Black"/>
+        <material value="Gazebo/Black"/>
     </gazebo>
     <gazebo reference="arm_5_link">
         <gravity>true</gravity>
         <self_collide>false</self_collide>
-        <material value="Schunk/LightGrey"/>
+        <material value="Gazebo/Grey"/>
     </gazebo>
     <gazebo reference="arm_6_link">
         <gravity>true</gravity>
         <self_collide>false</self_collide>
-        <material value="Schunk/Black"/>
+        <material value="Gazebo/Black"/>
     </gazebo>
     <gazebo reference="arm_7_link">
         <gravity>true</gravity>
         <self_collide>false</self_collide>
-        <material value="Schunk/LightGrey"/>
+        <material value="Gazebo/Grey"/>
     </gazebo>
 </robot>

File: src/mp500lwa4d_description/urdf/arm/arm.transmission.xacro (robot description, xacro)
@@ -9,5 +9,5 @@
             <actuator name="arm_${joint_num}_motor">
                 <hardwareInterface>hardware_interface/EffortJointInterface</hardwareInterface>
-                <mechanicalReduction>0.1</mechanicalReduction>
+                <mechanicalReduction>1</mechanicalReduction>
             </actuator>
         </transmission>

File: src/mp500lwa4d_description/urdf/arm/arm_lwa4d.urdf.xacro (robot description, xacro)
@@ -18,5 +18,5 @@
                     <mesh filename="package://mp500lwa4d_description/meshes/lwa4d/arm_podest_link.stl"/>
                 </geometry>
-                <material name="Schunk/LightGrey"/>
+                <material name="LightGrey"/>
             </visual>
             <collision>
@@ -55,9 +55,14 @@
                 <inertia ixx="0.001" ixy="0.0" ixz="0.0" iyy="0.001" iyz="0.0" izz="0.001" />
             </inertial>
+            <!--
+            <xacro:cylinder_inertial radius="0.06" length="0.150" mass="3.6">
+                <origin xyz="0 0 0.02" rpy="0 0 0"/>
+            </xacro:cylinder_inertial>
+            -->
             <visual>
                 <geometry>
                     <mesh filename="package://mp500lwa4d_description/meshes/lwa4d/arm_1_link.stl"/>
                 </geometry>
-                <material name="Schunk/LightGrey"/>
+                <material name="LightGrey"/>
             </visual>
             <collision>
@@ -82,9 +87,14 @@
                 <inertia ixx="0.001" ixy="0.0" ixz="0.0" iyy="0.001" iyz="0.0" izz="0.001" />
             </inertial>
+            <!--
+            <xacro:cylinder_inertial radius="0.06" length="0.150" mass="2.0">
+                <origin xyz="0 0 0" rpy="0 0 0"/>
+            </xacro:cylinder_inertial>
+            -->
             <visual>
                 <geometry>
                     <mesh filename="package://mp500lwa4d_description/meshes/lwa4d/arm_2_link.stl"/>
                 </geometry>
-                <material name="Schunk/Black"/>
+                <material name="Black"/>
             </visual>
             <collision>
@@ -109,9 +119,14 @@
                 <inertia ixx="0.001" ixy="0.0" ixz="0.0" iyy="0.001" iyz="0.0" izz="0.001" />
             </inertial>
+            <!--
+            <xacro:cylinder_inertial radius="0.06" length="0.2" mass="2.0">
+                <origin xyz="0.0 0 -0.2" rpy="0 0 0"/>
+            </xacro:cylinder_inertial>
+            -->
             <visual>
                 <geometry>
                     <mesh filename="package://mp500lwa4d_description/meshes/lwa4d/arm_3_link.stl"/>
                 </geometry>
-                <material name="Schunk/LightGrey"/>
+                <material name="LightGrey"/>
             </visual>
             <collision>
@@ -136,9 +151,14 @@
                 <inertia ixx="0.001" ixy="0.0" ixz="0.0" iyy="0.001" iyz="0.0" izz="0.001" />
             </inertial>
+            <!--
+            <xacro:cylinder_inertial radius="0.06" length="0.150" mass="1.2">
+                <origin xyz="0 0 0" rpy="0 0 0"/>
+            </xacro:cylinder_inertial>
+            -->
             <visual>
                 <geometry>
                     <mesh filename="package://mp500lwa4d_description/meshes/lwa4d/arm_4_link.stl"/>
                 </geometry>
-            <material name="Schunk/Black"/>
+            <material name="Black"/>
             </visual>
             <collision>
@@ -163,9 +183,14 @@
                 <inertia ixx="0.001" ixy="0.0" ixz="0.0" iyy="0.001" iyz="0.0" izz="0.001" />
             </inertial>
+            <!--
+            <xacro:cylinder_inertial radius="0.06" length="0.15" mass="1.2">
+                <origin xyz="0 0 -0.18" rpy="0 0 0"/>
+            </xacro:cylinder_inertial>
+            -->
             <visual>
                 <geometry>
                     <mesh filename="package://mp500lwa4d_description/meshes/lwa4d/arm_5_link.stl"/>
                 </geometry>
-                <material name="Schunk/LightGrey"/>
+                <material name="LightGrey"/>
             </visual>
             <collision>
@@ -181,5 +206,5 @@
             <parent link="arm_5_link"/>
             <child link="arm_6_link"/>
-            <limit effort="15" velocity="1.2566" lower="${-2.09 + safety_offset}" upper="${2.09 - safety_offset}"/>
+            <limit effort="15" velocity="1.2566" lower="${-2.96 + safety_offset}" upper="${2.96 - safety_offset}"/>
         </joint>
     <!-- arm_6_link -->
@@ -190,9 +215,14 @@
                 <inertia ixx="0.001" ixy="0.0" ixz="0.0" iyy="0.001" iyz="0.0" izz="0.001" />
             </inertial>
+            <!--
+            <xacro:sphere_inertial radius="0.05" mass="1.9">
+                <origin xyz="0 0 0" rpy="0 0 0"/>
+            </xacro:sphere_inertial>
+            -->
             <visual>
                 <geometry>
                     <mesh filename="package://mp500lwa4d_description/meshes/lwa4d/arm_6_link.stl"/>
                 </geometry>
-                <material name="Schunk/Black"/>
+                <material name="Black"/>
             </visual>
             <collision>
@@ -218,7 +248,7 @@
             </inertial>
             <!--
-                <xacro:cylinder_inertial radius="0.03" length="0.035" mass="0.05">
+            <xacro:cylinder_inertial radius="0.03" length="0.035" mass="0.05">
                 <origin xyz="0 0 0.06" rpy="0 0 0"/>
-                </xacro:cylinder_inertial>
+            </xacro:cylinder_inertial>
             -->
             <visual>
@@ -226,5 +256,5 @@
                     <mesh filename="package://mp500lwa4d_description/meshes/lwa4d/arm_7_link.stl"/>
                 </geometry>
-                <material name="Schunk/LightGrey"/>
+                <material name="LightGrey"/>
             </visual>
             <collision>
@@ -236,5 +266,4 @@
         <joint name="arm_ee_joint" type="fixed">
             <origin xyz="0 0 0.0824" rpy="0 0 0"/>
-            <axis xyz="0 0 1"/>
             <parent link="arm_7_link"/>
             <child link="arm_ee_link"/>

File: src/mp500lwa4d_description/urdf/base/base.gazebo.xacro (robot description, xacro)
@@ -13,4 +13,5 @@
           <kd>1.0</kd>
           <fdir1 value="1 0 0"/>
+          <material value="Gazebo/Grey"/>
       </gazebo>
       <!-- Right Wheel -->
@@ -22,4 +23,5 @@
           <kd>1.0</kd>
           <fdir1 value="1 0 0"/>
+          <material value="Gazebo/Grey"/>
       </gazebo>
       <!-- Castor -->
@@ -28,4 +30,5 @@
           <mu1>0.0</mu1>
           <mu2>0.0</mu2>
+          <material value="Gazebo/Grey"/>
       </gazebo>
       <gazebo reference="castor_front">
@@ -33,4 +36,5 @@
           <mu1>0.0</mu1>
           <mu2>0.0</mu2>
+          <material value="Gazebo/Grey"/>
       </gazebo>
 </robot>

File: src/mp500lwa4d_description/urdf/base/base_mp500.urdf.xacro (robot description, xacro)
@@ -19,5 +19,5 @@
 			<!--box size="0.445 0.277 0.17"/-->
 			</geometry>
-			<material name="Neobotix/Grey" />
+			<material name="Grey" />
 		</visual>
 		<collision name='body_collision'>
@@ -32,5 +32,5 @@
 	<link name="wheel_left_link" type="wheel">
 		<inertial>
-			<mass value="1.0" />
+			<mass value="1" />
 			<origin xyz="0 0 0" rpy="0 0 0" />
 			<inertia ixx="0.0045" ixy="0" ixz="0" iyy="0.0078" iyz="0" izz="0.0045" />
@@ -41,10 +41,10 @@
 				<mesh filename="package://mp500lwa4d_description/meshes/mp500/MP500-WHEEL.STL" scale="0.01 0.01 0.01" />
 			</geometry>
-			<material name="Neobotix/Black" />
+			<material name="Black" />
 		</visual>
 		<collision>
 			<origin xyz="0 0 0" rpy="0 1.57 -1.57" />
 			<geometry>
-				<cylinder radius="0.125" length="0.085"/>
+				<cylinder radius="0.13" length="0.085"/>
 		</geometry>
 		</collision>
@@ -54,5 +54,5 @@
 		<origin xyz="-0.155 0.255 0.13" rpy="0 0 0" />
 		<axis xyz="0 1 0"/>
-		<limit effort="10000.0" velocity="1.5"/>
+		<limit effort="11.3" velocity="1.5"/>
 		<joint_properties damping="0.0" friction="0.0" />
 		<parent link="base_link" />
@@ -100,10 +100,10 @@
 				<mesh filename="package://mp500lwa4d_description/meshes/mp500/MP500-WHEEL.STL" scale="0.01 0.01 0.01" />
 			</geometry>
-			<material name="Neobotix/Black" />
+			<material name="Black" />
 		</visual>
 		<collision>
 			<origin xyz="0 0 0" rpy="0 1.57 -1.57" />
 			<geometry>
-				<cylinder radius="0.125" length="0.085"/>
+				<cylinder radius="0.13" length="0.085"/>
 			</geometry>
 		</collision>
@@ -113,5 +113,5 @@
 		<origin xyz="-0.155 -0.255 0.13" rpy="0 0 0" />
 		<axis xyz="0 1 0"/>
-		<limit effort="10000.0" velocity="1.5"/>
+		<limit effort="11.3" velocity="1.5"/>
 		<joint_properties damping="0.0" friction="0.0" />
 		<parent link="base_link" />
@@ -130,5 +130,5 @@
 				<mesh filename="package://mp500lwa4d_description/meshes/mp500/HANGER-WHEEL.STL" scale="0.01 0.01 0.01" />
 			</geometry>
-			<material name="Neobotix/Grey" />
+			<material name="Grey" />
 		</visual>
 		<collision>
@@ -157,5 +157,5 @@
 				<sphere radius="0.005"/>
 			</geometry>
-			<material name="Neobotix/Grey" />
+			<material name="Grey" />
 		</visual>
 		<collision>

File: src/mp500lwa4d_description/urdf/common.xacro (robot description, xacro)
@@ -2,42 +2,36 @@
 <robot xmlns:xacro="http://www.ros.org/wiki/xacro">
     <!--+++++++++ Material +++++++++-->
-    <material name="Neobotix/Black">
+    <material name="Black">
         <color rgba="0.0 0.0 0.0 1.0"/>
     </material>
-    <material name="Neobotix/Blue">
+    <material name="Blue">
         <color rgba="0.0 0.0 0.8 1.0"/>
     </material>
-    <material name="Neobotix/Green">
+    <material name="Green">
         <color rgba="0.0 0.8 0.0 1.0"/>
     </material>
-    <material name="Neobotix/Grey">
+    <material name="Grey">
         <color rgba="0.7 0.7 0.7 1.0"/>
     </material>
-    <material name="Neobotix/Grey2">
+    <material name="Grey2">
         <color rgba="0.9 0.9 0.9 1.0"/>
     </material>
-    <material name="Neobotix/Red">
+    <material name="Red">
         <color rgba="0.8 0.0 0.0 1.0"/>
     </material>
-    <material name="Neobotix/White">
+    <material name="White">
         <color rgba="1.0 1.0 1.0 1.0"/>
     </material>
-    <material name="Neobotix/Yellow">
-        <color rgba="1.0 1.0 0 10" />
+    <material name="Yellow">
+        <color rgba="1.0 1.0 0 1.0" />
     </material>
-    <material name="Schunk/LightGrey">
+    <material name="LightGrey">
         <color rgba="0.7 0.7 0.7 1.0"/>
     </material>
-    <material name="Schunk/DarkGrey">
+    <material name="DarkGrey">
         <color rgba="0.4 0.4 0.4 1.0"/>
     </material>
-    <material name="Schunk/Black">
-        <color rgba="0.0 0.0 0.0 1.0"/>
-    </material>
-    <material name="Schunk/DarkGolden">
+    <material name="DarkGolden">
         <color rgba="0.4 0.4 0.3 1.0"/>
-    </material>
-    <material name="Schunk/Blue">
-        <color rgba="0.0 0.0 0.8 1.0"/>
     </material>
     <!--+++++++++ Property +++++++++-->

File: src/mp500lwa4d_description/urdf/robot.gazebo.xacro (robot description, xacro)
@@ -5,9 +5,9 @@
         <robotNamespace>/mp500lwa4d</robotNamespace>
         <alwaysOn>true</alwaysOn>
-        <updateRate>100</updateRate>
+        <updateRate>50</updateRate>
         <leftJoint>wheel_left_joint</leftJoint>
         <rightJoint>wheel_right_joint</rightJoint>
         <wheelSeparation>0.51</wheelSeparation>
-        <wheelDiameter>0.25</wheelDiameter>
+        <wheelDiameter>0.26</wheelDiameter>
         <torque>45</torque>
         <commandTopic>/mobile_base_controller/cmd_vel</commandTopic>
@@ -26,5 +26,5 @@
         <!--plugin name="ros_control" filename="libhwi_switch_gazebo_ros_control.so"-->
         <plugin name="gazebo_ros_control" filename="libgazebo_ros_control.so">
-            <robotNamespace>mp500lwa4d</robotNamespace>
+            <robotNamespace>/mp500lwa4d</robotNamespace>
             <filterJointsParam>joint_names</filterJointsParam>
         </plugin>

File: src/mp500lwa4d_description/urdf/sensor/rplidar.gazebo.xacro (robot description, xacro)
@@ -2,5 +2,5 @@
 <robot xmlns:xacro="http://www.ros.org/wiki/xacro">
     <gazebo reference="laserscanner_front_link">
-        <material>Neobotix/Yellow</material>
+        <material value="Gazebo/Grey"/>
     </gazebo>
     <gazebo reference="laserscanner_front_link">

File: src/mp500lwa4d_description/urdf/sensor/rplidar.urdf.xacro (robot description, xacro)
@@ -19,7 +19,7 @@
 				<geometry>
                 	<!--cylinder length="0.154" radius="0.053" /-->
-            		<mesh filename="package://neo_mp_500/robot_model/mp_500/meshes/SICK-S300.STL" />
+            		<mesh filename="package://mp500lwa4d_description/meshes/mp500/SICK-S300.STL" />
 				</geometry>
-				<material name="Neobotix/Yellow" />
+				<material name="Gazebo/Yellow" />
   			</visual>
   			<collision>

Commit message: debag gripper

File: src/mp500lwa4d_description/urdf/arm/arm.gazebo.xacro (robot description, xacro)
@@ -1,5 +1,4 @@
 <?xml version="1.0"?>
 <robot xmlns:xacro="http://www.ros.org/wiki/xacro">
-    <!--<xacro:include filename="$(find mp500lwa4d_description)/urdf/common.xacro" />-->
     <gazebo reference="arm_base_link">
         <gravity>true</gravity>

File: src/mp500lwa4d_description/urdf/arm/arm_lwa4d.urdf.xacro (robot description, xacro)
@@ -46,5 +46,5 @@
             <parent link="arm_base_link"/>
             <child link="arm_1_link"/>
-            <limit effort="216" velocity="0.43633" lower="${-M_PI+safety_offset}" upper="${M_PI-safety_offset}"/>
+            <limit effort="2160" velocity="0.43633" lower="${-M_PI+safety_offset}" upper="${M_PI-safety_offset}"/>
         </joint>
     <!-- arm_1_link-->
@@ -78,5 +78,5 @@
             <parent link="arm_1_link"/>
             <child link="arm_2_link"/>
-            <limit effort="216" velocity="0.43633" lower="${-2.14 + safety_offset}" upper="${2.14 - safety_offset}"/>
+            <limit effort="2160" velocity="0.43633" lower="${-2.14 + safety_offset}" upper="${2.14 - safety_offset}"/>
         </joint>
     <!-- arm_2_link -->
@@ -110,5 +110,5 @@
             <parent link="arm_2_link"/>
             <child link="arm_3_link"/>
-            <limit effort="81.5" velocity="0.4189" lower="${-M_PI + safety_offset}" upper="${M_PI - safety_offset}"/>
+            <limit effort="8150" velocity="0.4189" lower="${-M_PI + safety_offset}" upper="${M_PI - safety_offset}"/>
         </joint>
     <!-- arm_3_link -->
@@ -142,5 +142,5 @@
             <parent link="arm_3_link"/>
             <child link="arm_4_link"/>
-            <limit effort="81.5" velocity="0.4189" lower="${-2.18 + safety_offset}" upper="${2.18 - safety_offset}"/>
+            <limit effort="8150" velocity="0.4189" lower="${-2.18 + safety_offset}" upper="${2.18 - safety_offset}"/>
         </joint>
     <!--arm_4_link -->
@@ -174,5 +174,5 @@
             <parent link="arm_4_link"/>
             <child link="arm_5_link"/>
-            <limit effort="20.7" velocity="0.43633" lower="${-M_PI + safety_offset}" upper="${M_PI - safety_offset}"/>
+            <limit effort="2070" velocity="0.43633" lower="${-M_PI + safety_offset}" upper="${M_PI - safety_offset}"/>
         </joint>
     <!-- arm_5_link -->
@@ -206,5 +206,5 @@
             <parent link="arm_5_link"/>
             <child link="arm_6_link"/>
-            <limit effort="15" velocity="1.2566" lower="${-2.96 + safety_offset}" upper="${2.96 - safety_offset}"/>
+            <limit effort="1500" velocity="1.2566" lower="${-2.96 + safety_offset}" upper="${2.96 - safety_offset}"/>
         </joint>
     <!-- arm_6_link -->
@@ -238,5 +238,5 @@
             <parent link="arm_6_link"/>
             <child link="arm_7_link"/>
-            <limit effort="15" velocity="1.2566" lower="${-2.96 + safety_offset}" upper="${2.96 - safety_offset}"/>
+            <limit effort="1500" velocity="1.2566" lower="${-2.96 + safety_offset}" upper="${2.96 - safety_offset}"/>
         </joint>
     <!--arm_7_link -->
@@ -264,16 +264,4 @@
             </collision>
         </link>
-        <joint name="arm_ee_joint" type="fixed">
-            <origin xyz="0 0 0.0824" rpy="0 0 0"/>
-            <parent link="arm_7_link"/>
-            <child link="arm_ee_link"/>
-        </joint>
-        <link name="arm_ee_link">
-            <inertial>
-                <mass value="0.01" />
-                <origin xyz="0 0 0" />
-                <inertia ixx="0.001" ixy="0.0" ixz="0.0" iyy="0.001" iyz="0.0" izz="0.001" />
-            </inertial>
-        </link>
     </xacro:macro>
 </robot>

File: src/mp500lwa4d_description/urdf/base/base.gazebo.xacro (robot description, xacro)
@@ -32,9 +32,11 @@
       <gazebo reference="hanger">
           <gravity>true</gravity>
-          <mu1>0.0</mu1>
-          <mu2>0.0</mu2>
+          <mu1>0.1</mu1>
+          <mu2>0.1</mu2>
+          <kp>1000000.0</kp>
+          <kd>100.0</kd>
           <material value="Gazebo/Grey"/>
       </gazebo>
-      <gazebo reference="castor_front">
+      <!--<gazebo reference="castor_front">
           <gravity>true</gravity>
           <mu1>0.1</mu1>
@@ -43,4 +45,4 @@
           <kd>100.0</kd>
           <material value="Gazebo/Grey"/>
-      </gazebo>
+      </gazebo>-->
 </robot>

File: src/mp500lwa4d_description/urdf/base/base_mp500.urdf.xacro (robot description, xacro)
@@ -18,7 +18,9 @@
 	<link name="base_link">
 		<inertial>
-			<mass value="25.67" />
+			<mass value="100"/>
+        	<inertia ixx="0.5" ixy="0" ixz="0" iyy="0.5" iyz="0" izz="0.5" />
+			<!--<mass value="25.67" />
 			<origin xyz="0 0 0.216" rpy="0 0 0"/>
-			<inertia ixx="0.54" ixy="0.0" ixz="0.0" iyy="1.08" iyz="0.0" izz="1.23" />
+			<inertia ixx="0.54" ixy="0.0" ixz="0.0" iyy="1.08" iyz="0.0" izz="1.23" />-->
 		</inertial>
 		<visual name='body'>
@@ -148,5 +150,5 @@
 			<origin xyz="0 0 0" rpy="0 0 -1.57" />
 			<geometry>
-				<sphere radius="0.00115"/>
+				<mesh filename="package://mp500lwa4d_description/meshes/mp500/HANGER-WHEEL.STL" scale="0.01 0.01 0.01" />
 			</geometry>
 		</collision>
@@ -159,5 +161,5 @@
 	</joint>
 <!--+++++++++++++++ castor_front +++++++++++++++-->
-	<link name="castor_front">
+	<!--<link name="castor_front">
 		<inertial>
 			<mass value="0.001" />
@@ -184,4 +186,4 @@
 		<parent link="base_link" />
 		<child link="castor_front" />
-	</joint>
+	</joint>-->
 </robot>

File: src/mp500lwa4d_description/urdf/robot.gazebo.xacro (robot description, xacro)
@@ -27,5 +27,4 @@
         <plugin name="gazebo_ros_control" filename="libgazebo_ros_control.so">
             <robotNamespace>/mp500lwa4d</robotNamespace>
-            <robotBaseFrame>base_footprint</robotBaseFrame>
         </plugin>
     </gazebo>

File: src/mp500lwa4d_description/urdf/robot.urdf.xacro (robot description, xacro)
@@ -8,4 +8,6 @@
     <xacro:include filename="$(find mp500lwa4d_description)/urdf/arm/arm_lwa4d.urdf.xacro" />
     <xacro:arm_lwa4d parent="base_link"/>
+    <xacro:include filename="$(find mp500lwa4d_description)/urdf/gripper/gripper_pg70.urdf.xacro" />
+    <xacro:gripper_pg70 parent="arm_7_link" has_podest="1"/>
     <xacro:include filename="$(find mp500lwa4d_description)/urdf/sensor/rplidar.urdf.xacro" />
     <xacro:laser parent="base_link"/>
@@ -13,8 +15,10 @@
     <xacro:include filename="$(find mp500lwa4d_description)/urdf/base/base.gazebo.xacro" />
     <xacro:include filename="$(find mp500lwa4d_description)/urdf/arm/arm.gazebo.xacro" />
+    <xacro:include filename="$(find mp500lwa4d_description)/urdf/gripper/gripper.gazebo.xacro" />
     <xacro:include filename="$(find mp500lwa4d_description)/urdf/sensor/rplidar.gazebo.xacro" />
     <!--++++++++++ Transmission +++++++++++-->
     <xacro:include filename="$(find mp500lwa4d_description)/urdf/base/base.transmission.xacro" />
     <xacro:include filename="$(find mp500lwa4d_description)/urdf/arm/arm.transmission.xacro" />
+    <xacro:include filename="$(find mp500lwa4d_description)/urdf/gripper/gripper.transmission.xacro" />
     <!--+++++++++ ros controller +++++++++++-->
     <xacro:include filename="$(find mp500lwa4d_description)/urdf/robot.gazebo.xacro" />
