Commit message: fix arm vibration

File: src/mp500lwa4d_description/urdf/arm/arm_lwa4d.urdf.xacro (robot description, xacro)
@@ -46,5 +46,6 @@
             <parent link="arm_base_link"/>
             <child link="arm_1_link"/>
-            <limit effort="2160" velocity="0.43633" lower="${-M_PI+safety_offset}" upper="${M_PI-safety_offset}"/>
+            <limit effort="216" velocity="0.43633" lower="${-M_PI+safety_offset}" upper="${M_PI-safety_offset}"/>
+            <dynamics damping="0.0" friction="0.0"/>
         </joint>
     <!-- arm_1_link-->
@@ -78,5 +79,6 @@
             <parent link="arm_1_link"/>
             <child link="arm_2_link"/>
-            <limit effort="2160" velocity="0.43633" lower="${-2.14 + safety_offset}" upper="${2.14 - safety_offset}"/>
+            <limit effort="216" velocity="0.43633" lower="${-2.14 + safety_offset}" upper="${2.14 - safety_offset}"/>
+            <dynamics damping="0.9" friction="0.08"/>
         </joint>
     <!-- arm_2_link -->
@@ -110,5 +112,6 @@
             <parent link="arm_2_link"/>
             <child link="arm_3_link"/>
-            <limit effort="8150" velocity="0.4189" lower="${-M_PI + safety_offset}" upper="${M_PI - safety_offset}"/>
+            <limit effort="81.5" velocity="0.4189" lower="${-M_PI + safety_offset}" upper="${M_PI - safety_offset}"/>
+            <dynamics damping="0.0" friction="0.0"/>
         </joint>
     <!-- arm_3_link -->
@@ -142,5 +145,6 @@
             <parent link="arm_3_link"/>
             <child link="arm_4_link"/>
-            <limit effort="8150" velocity="0.4189" lower="${-2.18 + safety_offset}" upper="${2.18 - safety_offset}"/>
+            <limit effort="81.5" velocity="0.4189" lower="${-2.18 + safety_offset}" upper="${2.18 - safety_offset}"/>
+            <dynamics damping="0.9" friction="0.08"/>
         </joint>
     <!--arm_4_link -->
@@ -174,5 +178,6 @@
             <parent link="arm_4_link"/>
             <child link="arm_5_link"/>
-            <limit effort="2070" velocity="0.43633" lower="${-M_PI + safety_offset}" upper="${M_PI - safety_offset}"/>
+            <limit effort="20.7" velocity="0.43633" lower="${-M_PI + safety_offset}" upper="${M_PI - safety_offset}"/>
+            <dynamics damping="0.0" friction="0.0"/>
         </joint>
     <!-- arm_5_link -->
@@ -206,5 +211,6 @@
             <parent link="arm_5_link"/>
             <child link="arm_6_link"/>
-            <limit effort="1500" velocity="1.2566" lower="${-2.96 + safety_offset}" upper="${2.96 - safety_offset}"/>
+            <limit effort="15" velocity="1.2566" lower="${-2.96 + safety_offset}" upper="${2.96 - safety_offset}"/>
+            <dynamics damping="0.0" friction="0.0"/>
         </joint>
     <!-- arm_6_link -->
@@ -238,5 +244,5 @@
             <parent link="arm_6_link"/>
             <child link="arm_7_link"/>
-            <limit effort="1500" velocity="1.2566" lower="${-2.96 + safety_offset}" upper="${2.96 - safety_offset}"/>
+            <limit effort="15" velocity="1.2566" lower="${-2.96 + safety_offset}" upper="${2.96 - safety_offset}"/>
         </joint>
     <!--arm_7_link -->

File: src/mp500lwa4d_description/urdf/base/base.gazebo.xacro (robot description, xacro)
@@ -6,5 +6,5 @@
       </gazebo>
       <gazebo reference="base_link">
-          <gravity>false</gravity>
+          <gravity>true</gravity>
           <material value="Gazebo/Grey"/>
       </gazebo>

File: src/mp500lwa4d_description/urdf/gripper/gripper.gazebo.xacro (robot description, xacro)
@@ -2,20 +2,20 @@
 <robot xmlns:xacro="http://www.ros.org/wiki/xacro">
     <gazebo reference="gripper_podest_link">
-      <gravity>false</gravity>
+      <gravity>true</gravity>
       <self_collide>false</self_collide>
       <material>Gazebo/Black</material>
     </gazebo>
     <gazebo reference="gripper_palm_link">
-      <gravity>false</gravity>
-      <self_collide>false</self_collide>
+      <gravity>true</gravity>
+      <self_collide>true</self_collide>
       <material>Gazebo/Black</material>
     </gazebo>
     <gazebo reference="gripper_finger_left_link">
-      <gravity>false</gravity>
+      <gravity>true</gravity>
       <self_collide>false</self_collide>
       <material>Gazebo/Grey</material>
     </gazebo>
     <gazebo reference="gripper_finger_right_link">
-      <gravity>false</gravity>
+      <gravity>true</gravity>
       <self_collide>false</self_collide>
       <material>Gazebo/Grey</material>

File: src/mp500lwa4d_description/urdf/gripper/gripper_pg70.urdf.xacro (robot description, xacro)
@@ -67,4 +67,5 @@
       <axis xyz="0 1 0" />
       <limit effort="10" lower="-0.0301" upper="-0.005" velocity="0.041"/>
+      <dynamics damping="0.08" friction="0.08"/>
     </joint>
     <link name="gripper_finger_left_link">
@@ -95,4 +96,5 @@
       <!--<mimic joint="gripper_finger_left_joint" multiplier="1" offset="0"/>-->
       <limit effort="10" lower="0.005" upper="0.0301" velocity="0.041"/>
+      <dynamics damping="0.08" friction="0.08"/>
     </joint>
     <link name="gripper_finger_right_link">
