Commit message: reduce mess of base link to prevent base slipping

File: src/mp500lwa4d_description/urdf/base/base_mp500.urdf.xacro (robot description, xacro)
@@ -18,7 +18,8 @@
 	<link name="base_link">
 		<inertial>
-			<mass value="25.67" />
+			<mass value="1" />
 			<origin xyz="0 0 0.216" rpy="0 0 0"/>
-			<inertia ixx="0.54" ixy="0.0" ixz="0.0" iyy="1.08" iyz="0.0" izz="1.23" />
+			<!--<inertia ixx="0.54" ixy="0.0" ixz="0.0" iyy="1.08" iyz="0.0" izz="1.23" />-->
+			<inertia ixx="1" ixy="0.0" ixz="0.0" iyy="1" iyz="0.0" izz="1" />
 		</inertial>
 		<visual name='body'>
@@ -148,5 +149,5 @@
 			<origin xyz="0 0 0" rpy="0 0 -1.57" />
 			<geometry>
-				<sphere radius="0.00115"/>
+				<mesh filename="package://mp500lwa4d_description/meshes/mp500/HANGER-WHEEL.STL" scale="0.01 0.01 0.01" />
 			</geometry>
 		</collision>
@@ -159,4 +160,5 @@
 	</joint>
 <!--+++++++++++++++ castor_front +++++++++++++++-->
+<!--
 	<link name="castor_front">
 		<inertial>
@@ -184,4 +186,4 @@
 		<parent link="base_link" />
 		<child link="castor_front" />
-	</joint>
+	</joint>-->
 </robot>

Commit message: add moveit_cartesian_controller.py

File: src/mp500lwa4d_description/urdf/base/base_mp500.urdf.xacro (robot description, xacro)
@@ -19,5 +19,5 @@
 		<inertial>
 			<mass value="1" />
-			<origin xyz="0 0 0.216" rpy="0 0 0"/>
+			<!--<origin xyz="0 0 0.216" rpy="0 0 0"/>-->
 			<!--<inertia ixx="0.54" ixy="0.0" ixz="0.0" iyy="1.08" iyz="0.0" izz="1.23" />-->
 			<inertia ixx="1" ixy="0.0" ixz="0.0" iyy="1" iyz="0.0" izz="1" />

File: src/mp500lwa4d_description/urdf/robot.gazebo.xacro (robot description, xacro)
@@ -2,4 +2,8 @@
 <robot xmlns:xacro="http://www.ros.org/wiki/xacro">
     <gazebo>
+        <plugin name="gazebo_ros_control" filename="libgazebo_ros_control.so">
+            <robotNamespace>/mp500lwa4d</robotNamespace>
+            <robotBaseFrame>base_footprint</robotBaseFrame>
+        </plugin>
         <plugin name="differential_drive_controller" filename="libgazebo_ros_diff_drive.so">
         <robotNamespace>/mp500lwa4d</robotNamespace>
@@ -25,8 +29,4 @@
         </plugin>
         <!--plugin name="ros_control" filename="libhwi_switch_gazebo_ros_control.so"-->
-        <plugin name="gazebo_ros_control" filename="libgazebo_ros_control.so">
-            <robotNamespace>/mp500lwa4d</robotNamespace>
-            <robotBaseFrame>base_footprint</robotBaseFrame>
-        </plugin>
     </gazebo>
   </robot>

Commit message: fix git problem

File: src/mp500lwa4d_description/urdf/base/base_mp500.urdf.xacro (robot description, xacro)
@@ -18,16 +18,8 @@
 	<link name="base_link">
 		<inertial>
-<<<<<<< HEAD
 			<mass value="1" />
 			<!--<origin xyz="0 0 0.216" rpy="0 0 0"/>-->
 			<!--<inertia ixx="0.54" ixy="0.0" ixz="0.0" iyy="1.08" iyz="0.0" izz="1.23" />-->
 			<inertia ixx="1" ixy="0.0" ixz="0.0" iyy="1" iyz="0.0" izz="1" />
-=======
-			<mass value="100"/>
-        	<inertia ixx="0.5" ixy="0" ixz="0" iyy="0.5" iyz="0" izz="0.5" />
-			<!--<mass value="25.67" />
-			<origin xyz="0 0 0.216" rpy="0 0 0"/>
-			<inertia ixx="0.54" ixy="0.0" ixz="0.0" iyy="1.08" iyz="0.0" izz="1.23" />-->
->>>>>>> Debug
 		</inertial>
 		<visual name='body'>
@@ -167,35 +159,3 @@
 		<child link="hanger" />
 	</joint>
-<!--+++++++++++++++ castor_front +++++++++++++++-->
-<<<<<<< HEAD
-<!--
-	<link name="castor_front">
-=======
-	<!--<link name="castor_front">
->>>>>>> Debug
-		<inertial>
-			<mass value="0.001" />
-			<origin xyz="0 0 0" rpy="0 0 0" />
-			<inertia ixx="0.000025" ixy="0" ixz="0" iyy="0.000025" iyz="0" izz="0.000025" />
-		</inertial>
-		<visual>
-			<origin xyz="0 0 0" rpy="0 0 0" />
-			<geometry>
-				<sphere radius="0.005"/>
-			</geometry>
-			<material name="Grey" />
-		</visual>
-		<collision>
-			<origin xyz="0 0 0" rpy="0 0 0" />
-			<geometry>
-				<sphere radius="0.005"/>
-			</geometry>
-		</collision>
-	</link>
-	<joint name="castor_front_joint" type="fixed">
-		<origin xyz="0.3 0 0.01" rpy="0 0 0"/>
-		<axis xyz="0 0 1"/>
-		<parent link="base_link" />
-		<child link="castor_front" />
-	</joint>-->
 </robot>

File: src/mp500lwa4d_description/urdf/robot.gazebo.xacro (robot description, xacro)
@@ -29,10 +29,4 @@
         </plugin>
         <!--plugin name="ros_control" filename="libhwi_switch_gazebo_ros_control.so"-->
-<<<<<<< HEAD
-=======
-        <plugin name="gazebo_ros_control" filename="libgazebo_ros_control.so">
-            <robotNamespace>/mp500lwa4d</robotNamespace>
-        </plugin>
->>>>>>> Debug
     </gazebo>
   </robot>

Commit message: add RL env. and DDPG algorithm

File: src/mp500lwa4d_description/urdf/base/base_mp500.urdf.xacro (robot description, xacro)
@@ -61,5 +61,5 @@
 			<geometry>
 				<cylinder radius="0.125" length="0.085"/>
-		</geometry>
+			</geometry>
 		</collision>
 	</link>
