Commit message: fix problems

File: src/mp500lwa4d_description/urdf/base/base.gazebo.xacro (robot description, xacro)
@@ -3,12 +3,12 @@
       <!-- Base Link -->
       <gazebo reference="base_link">
-          <turnGravityOff>false</turnGravityOff>
+          <gravity>true</gravity>
       </gazebo>
       <!-- Left Wheel -->
       <gazebo reference="wheel_left_link">
-          <turnGravityOff>false</turnGravityOff>
-          <mu1>1.0</mu1>
-          <mu2>1.0</mu2>
-          <kp>10000000.0</kp>
+          <gravity>true</gravity>
+          <mu1>1000.0</mu1>
+          <mu2>500.0</mu2>
+          <kp>1000000.0</kp>
           <kd>1.0</kd>
           <fdir1 value="1 0 0"/>
@@ -17,8 +17,8 @@
       <!-- Right Wheel -->
       <gazebo reference="wheel_right_link">
-          <turnGravityOff>false</turnGravityOff>
-          <mu1>1.0</mu1>
-          <mu2>1.0</mu2>
-          <kp>10000000.0</kp>
+          <gravity>true</gravity>
+          <mu1>1000.0</mu1>
+          <mu2>500.0</mu2>
+          <kp>1000000.0</kp>
           <kd>1.0</kd>
           <fdir1 value="1 0 0"/>
@@ -27,5 +27,5 @@
       <!-- Castor -->
       <gazebo reference="hanger">
-          <turnGravityOff>false</turnGravityOff>
+          <gravity>true</gravity>
           <mu1>0.0</mu1>
           <mu2>0.0</mu2>
@@ -33,5 +33,5 @@
       </gazebo>
       <gazebo reference="castor_front">
-          <turnGravityOff>false</turnGravityOff>
+          <gravity>true</gravity>
           <mu1>0.0</mu1>
           <mu2>0.0</mu2>

File: src/mp500lwa4d_description/urdf/base/base.transmission.xacro (robot description, xacro)
@@ -9,5 +9,5 @@
             <actuator name="wheel_${joint_loc}_motor">
                 <hardwareInterface>hardware_interface/EffortJointInterface</hardwareInterface>
-                <mechanicalReduction>0.1</mechanicalReduction>
+                <mechanicalReduction>1</mechanicalReduction>
             </actuator>
         </transmission>

File: src/mp500lwa4d_description/urdf/base/base_mp500.urdf.xacro (robot description, xacro)
@@ -167,5 +167,5 @@
 	</link>
 	<joint name="castor_front_joint" type="fixed">
-		<origin xyz="0.3 0 0.01" rpy="0 0 0"/>
+		<origin xyz="0.3 0 0.014" rpy="0 0 0"/>
 		<axis xyz="0 0 1"/>
 		<parent link="base_link" />

File: src/mp500lwa4d_description/urdf/robot.gazebo.xacro (robot description, xacro)
@@ -13,11 +13,11 @@
         <commandTopic>/mobile_base_controller/cmd_vel</commandTopic>
         <odometryTopic>odom</odometryTopic>
-        <odometryFrame>map</odometryFrame>
-        <robotBaseFrame>/mp500lwa4d/base_link</robotBaseFrame>
+        <odometryFrame>odom</odometryFrame>
+        <robotBaseFrame>base_link</robotBaseFrame>
         <legacyMode>false</legacyMode>
         <rosDebugLevel>Debug</rosDebugLevel>
         <publishWheelTF>true</publishWheelTF>
         <publishWheelJointState>true</publishWheelJointState>
-        <wheelAcceleration>0.01</wheelAcceleration>
+        <wheelAcceleration>2.4</wheelAcceleration>
         <wheelTorque>50</wheelTorque>
         <publishTf>1</publishTf>

Commit message: catkin_make

File: src/mp500lwa4d_description/urdf/base/base.gazebo.xacro (robot description, xacro)
@@ -2,14 +2,18 @@
 <robot xmlns:xacro="http://www.ros.org/wiki/xacro">
       <!-- Base Link -->
+      <gazebo reference="base_footprint">
+          <material value="Gazebo/Grey"/>
+      </gazebo>
       <gazebo reference="base_link">
-          <gravity>true</gravity>
+          <gravity>false</gravity>
+          <material value="Gazebo/Grey"/>
       </gazebo>
       <!-- Left Wheel -->
       <gazebo reference="wheel_left_link">
           <gravity>true</gravity>
-          <mu1>1000.0</mu1>
-          <mu2>500.0</mu2>
+          <mu1>100.5</mu1>
+          <mu2>100.5</mu2>
           <kp>1000000.0</kp>
-          <kd>1.0</kd>
+          <kd>100.0</kd>
           <fdir1 value="1 0 0"/>
           <material value="Gazebo/Grey"/>
@@ -18,8 +22,8 @@
       <gazebo reference="wheel_right_link">
           <gravity>true</gravity>
-          <mu1>1000.0</mu1>
-          <mu2>500.0</mu2>
+          <mu1>100.5</mu1>
+          <mu2>100.5</mu2>
           <kp>1000000.0</kp>
-          <kd>1.0</kd>
+          <kd>100.0</kd>
           <fdir1 value="1 0 0"/>
           <material value="Gazebo/Grey"/>

File: src/mp500lwa4d_description/urdf/base/base_mp500.urdf.xacro (robot description, xacro)
@@ -3,4 +3,17 @@
        name="base_mp500" >
 <!--++++++++++++++++++base_link+++++++++++++++++++++-->
+	<joint name="base_footprint_joint" type="fixed">
+		<origin xyz="0 0 0" rpy="0 0 0" />
+		<parent link="base_footprint"/>
+		<child link="base_link" />
+	</joint>
+	<link name="base_footprint">
+		<visual>
+			<origin xyz="0 0 0" rpy="0 0 0" />
+			<geometry>
+				<box size="0.001 0.001 0.001" />
+			</geometry>
+		</visual>
+	</link>
 	<link name="base_link">
 		<inertial>
@@ -54,6 +67,6 @@
 		<origin xyz="-0.155 0.255 0.13" rpy="0 0 0" />
 		<axis xyz="0 1 0"/>
-		<limit effort="11.3" velocity="1.5"/>
-		<joint_properties damping="0.0" friction="0.0" />
+		<limit effort="20" velocity="1.5"/>
+		<dynamics damping="0.0" friction="0.0" />
 		<parent link="base_link" />
 		<child link="wheel_left_link" />
@@ -113,6 +126,6 @@
 		<origin xyz="-0.155 -0.255 0.13" rpy="0 0 0" />
 		<axis xyz="0 1 0"/>
-		<limit effort="11.3" velocity="1.5"/>
-		<joint_properties damping="0.0" friction="0.0" />
+		<limit effort="20" velocity="1.5"/>
+		<dynamics damping="0.0" friction="0.0" />
 		<parent link="base_link" />
 		<child link="wheel_right_link" />
@@ -167,5 +180,5 @@
 	</link>
 	<joint name="castor_front_joint" type="fixed">
-		<origin xyz="0.3 0 0.014" rpy="0 0 0"/>
+		<origin xyz="0.3 0 0.01" rpy="0 0 0"/>
 		<axis xyz="0 0 1"/>
 		<parent link="base_link" />

File: src/mp500lwa4d_description/urdf/robot.gazebo.xacro (robot description, xacro)
@@ -10,15 +10,15 @@
         <wheelSeparation>0.51</wheelSeparation>
         <wheelDiameter>0.26</wheelDiameter>
-        <torque>45</torque>
+        <torque>30</torque>
         <commandTopic>/mobile_base_controller/cmd_vel</commandTopic>
         <odometryTopic>odom</odometryTopic>
         <odometryFrame>odom</odometryFrame>
-        <robotBaseFrame>base_link</robotBaseFrame>
+        <robotBaseFrame>base_footprint</robotBaseFrame>
         <legacyMode>false</legacyMode>
         <rosDebugLevel>Debug</rosDebugLevel>
         <publishWheelTF>true</publishWheelTF>
         <publishWheelJointState>true</publishWheelJointState>
-        <wheelAcceleration>2.4</wheelAcceleration>
-        <wheelTorque>50</wheelTorque>
+        <wheelAcceleration>0.01</wheelAcceleration>
+        <wheelTorque>30</wheelTorque>
         <publishTf>1</publishTf>
         <odometrySource>encoder</odometrySource>
@@ -27,5 +27,5 @@
         <plugin name="gazebo_ros_control" filename="libgazebo_ros_control.so">
             <robotNamespace>/mp500lwa4d</robotNamespace>
-            <robotBaseFrame>base_link</robotBaseFrame>
+            <robotBaseFrame>base_footprint</robotBaseFrame>
         </plugin>
     </gazebo>

Commit message: fixed the friction probem of the wheel.

File: src/mp500lwa4d_description/urdf/base/base.gazebo.xacro (robot description, xacro)
@@ -12,9 +12,9 @@
       <gazebo reference="wheel_left_link">
           <gravity>true</gravity>
-          <mu1>100.5</mu1>
-          <mu2>100.5</mu2>
+          <mu1>1.5</mu1>
+          <mu2>1.5</mu2>
           <kp>1000000.0</kp>
           <kd>100.0</kd>
-          <fdir1 value="1 0 0"/>
+          <fdir1>0 0 1</fdir1>
           <material value="Gazebo/Grey"/>
       </gazebo>
@@ -22,9 +22,9 @@
       <gazebo reference="wheel_right_link">
           <gravity>true</gravity>
-          <mu1>100.5</mu1>
-          <mu2>100.5</mu2>
+          <mu1>1.5</mu1>
+          <mu2>1.5</mu2>
           <kp>1000000.0</kp>
           <kd>100.0</kd>
-          <fdir1 value="1 0 0"/>
+          <fdir1>0 0 1</fdir1>
           <material value="Gazebo/Grey"/>
       </gazebo>
@@ -40,4 +40,6 @@
           <mu1>0.0</mu1>
           <mu2>0.0</mu2>
+          <kp>1000000.0</kp>
+          <kd>100.0</kd>
           <material value="Gazebo/Grey"/>
       </gazebo>

File: src/mp500lwa4d_description/urdf/base/base_mp500.urdf.xacro (robot description, xacro)
@@ -59,5 +59,5 @@
 			<origin xyz="0 0 0" rpy="0 1.57 -1.57" />
 			<geometry>
-				<cylinder radius="0.13" length="0.085"/>
+				<cylinder radius="0.125" length="0.085"/>
 		</geometry>
 		</collision>
@@ -118,5 +118,5 @@
 			<origin xyz="0 0 0" rpy="0 1.57 -1.57" />
 			<geometry>
-				<cylinder radius="0.13" length="0.085"/>
+				<cylinder radius="0.125" length="0.085"/>
 			</geometry>
 		</collision>

File: src/mp500lwa4d_description/urdf/robot.gazebo.xacro (robot description, xacro)
@@ -9,5 +9,5 @@
         <rightJoint>wheel_right_joint</rightJoint>
         <wheelSeparation>0.51</wheelSeparation>
-        <wheelDiameter>0.26</wheelDiameter>
+        <wheelDiameter>0.25</wheelDiameter>
         <torque>30</torque>
         <commandTopic>/mobile_base_controller/cmd_vel</commandTopic>

Commit message: add base_move_controller.py, which can control robot move to a appointed point.

File: src/mp500lwa4d_description/urdf/base/base.gazebo.xacro (robot description, xacro)
@@ -12,6 +12,6 @@
       <gazebo reference="wheel_left_link">
           <gravity>true</gravity>
-          <mu1>1.5</mu1>
-          <mu2>1.5</mu2>
+          <mu1>100.5</mu1>
+          <mu2>100.5</mu2>
           <kp>1000000.0</kp>
           <kd>100.0</kd>
@@ -22,6 +22,6 @@
       <gazebo reference="wheel_right_link">
           <gravity>true</gravity>
-          <mu1>1.5</mu1>
-          <mu2>1.5</mu2>
+          <mu1>100.5</mu1>
+          <mu2>100.5</mu2>
           <kp>1000000.0</kp>
           <kd>100.0</kd>
@@ -38,6 +38,6 @@
       <gazebo reference="castor_front">
           <gravity>true</gravity>
-          <mu1>0.0</mu1>
-          <mu2>0.0</mu2>
+          <mu1>0.1</mu1>
+          <mu2>0.1</mu2>
           <kp>1000000.0</kp>
           <kd>100.0</kd>

File: src/mp500lwa4d_description/urdf/base/base_mp500.urdf.xacro (robot description, xacro)
@@ -67,5 +67,5 @@
 		<origin xyz="-0.155 0.255 0.13" rpy="0 0 0" />
 		<axis xyz="0 1 0"/>
-		<limit effort="20" velocity="1.5"/>
+		<limit effort="500" velocity="5"/>
 		<dynamics damping="0.0" friction="0.0" />
 		<parent link="base_link" />
@@ -126,5 +126,5 @@
 		<origin xyz="-0.155 -0.255 0.13" rpy="0 0 0" />
 		<axis xyz="0 1 0"/>
-		<limit effort="20" velocity="1.5"/>
+		<limit effort="500" velocity="5"/>
 		<dynamics damping="0.0" friction="0.0" />
 		<parent link="base_link" />

File: src/mp500lwa4d_description/urdf/robot.gazebo.xacro (robot description, xacro)
@@ -10,5 +10,5 @@
         <wheelSeparation>0.51</wheelSeparation>
         <wheelDiameter>0.25</wheelDiameter>
-        <torque>30</torque>
+        <torque>100</torque>
         <commandTopic>/mobile_base_controller/cmd_vel</commandTopic>
         <odometryTopic>odom</odometryTopic>
@@ -19,6 +19,6 @@
         <publishWheelTF>true</publishWheelTF>
         <publishWheelJointState>true</publishWheelJointState>
-        <wheelAcceleration>0.01</wheelAcceleration>
-        <wheelTorque>30</wheelTorque>
+        <wheelAcceleration>10</wheelAcceleration>
+        <wheelTorque>100</wheelTorque>
         <publishTf>1</publishTf>
         <odometrySource>encoder</odometrySource>

Commit message: fixed some physical problems. Add a mutilprocess version.

File: src/mp500lwa4d_description/urdf/base/base.gazebo.xacro (robot description, xacro)
@@ -36,4 +36,5 @@
           <kp>1000000.0</kp>
           <kd>100.0</kd>
+          <fdir1>0 0 1</fdir1>
           <material value="Gazebo/Grey"/>
       </gazebo>

File: src/mp500lwa4d_description/urdf/base/base_mp500.urdf.xacro (robot description, xacro)
@@ -31,5 +31,5 @@
 				<mesh filename="package://mp500lwa4d_description/meshes/mp500/MP500-BODY.STL" scale="0.01 0.01 0.01"/>
 			<!--cylinder length="0.381" radius="0.2545"/-->
-			<!--box size="0.445 0.277 0.17"/-->
+				<!--<box size="0.445 0.277 0.17"/>-->
 			</geometry>
 			<material name="Grey" />
@@ -38,4 +38,5 @@
 			<origin xyz="0 0 0.216" rpy="0 0 -1.57" />
 			<geometry>
+				<!--<mesh filename="package://mp500lwa4d_description/meshes/mp500/MP500-BODY.STL" scale="0.01 0.01 0.01"/>-->
 				<box size="0.400 0.676 0.300"/>
 				<!--cylinder length="0.381" radius="0.2545"/-->
@@ -46,5 +47,5 @@
 	<link name="wheel_left_link" type="wheel">
 		<inertial>
-			<mass value="1" />
+			<mass value="5" />
 			<origin xyz="0 0 0" rpy="0 0 0" />
 			<inertia ixx="0.0045" ixy="0" ixz="0" iyy="0.0078" iyz="0" izz="0.0045" />
@@ -104,5 +105,5 @@
 	<link name="wheel_right_link" type="wheel">
 		<inertial>
-			<mass value="1" />
+			<mass value="5" />
 			<origin xyz="0 0 0" rpy="0 0 0" />
 			<!--inertia ixx="0.0051" ixy="0" ixz="0" iyy="0.0051" iyz="0" izz="0.009" /-->
@@ -135,5 +136,5 @@
 	<link name="hanger">
 		<inertial>
-			<mass value="0.01" />
+			<mass value="5" />
 			<origin xyz="0 0 0" rpy="0 0 0" />
 			<inertia ixx="0.0013" ixy="0" ixz="0" iyy="0.0013" iyz="0" izz="0.0013" />

File: src/mp500lwa4d_description/urdf/goal.xacro (robot description, xacro)
@@ -8,7 +8,7 @@
     <link name="Goal">
         <inertial>
-			<mass value="1" />
+			<!--<mass value="0" />-->
 			<origin xyz="0 0 0" rpy="0 0 0" />
-			<inertia ixx="1" ixy="0" ixz="0" iyy="1" iyz="0" izz="1" />
+			<!--<inertia ixx="1" ixy="0" ixz="0" iyy="1" iyz="0" izz="1" />-->
 		</inertial>
         <visual>
@@ -22,5 +22,5 @@
     <gazebo reference="Goal">
           <material value="Gazebo/Red"/>
-          <gravity>False</gravity>
+          <gravity>0 0 0</gravity>
     </gazebo>
 </robot>

File: src/mp500lwa4d_description/urdf/robot.gazebo.xacro (robot description, xacro)
@@ -3,9 +3,9 @@
     <gazebo>
         <plugin name="gazebo_ros_control" filename="libgazebo_ros_control.so">
-            <robotNamespace>/mp500lwa4d</robotNamespace>
+            <!--<robotNamespace>mp500lwa4d</robotNamespace>-->
             <robotBaseFrame>base_footprint</robotBaseFrame>
         </plugin>
         <plugin name="differential_drive_controller" filename="libgazebo_ros_diff_drive.so">
-        <robotNamespace>/mp500lwa4d</robotNamespace>
+        <!--<robotNamespace>mp500lwa4d</robotNamespace>		  -->
         <alwaysOn>true</alwaysOn>
         <updateRate>50</updateRate>
@@ -15,5 +15,5 @@
         <wheelDiameter>0.25</wheelDiameter>
         <torque>100</torque>
-        <commandTopic>/mobile_base_controller/cmd_vel</commandTopic>
+        <commandTopic>mobile_base_controller/cmd_vel</commandTopic>
         <odometryTopic>odom</odometryTopic>
         <odometryFrame>odom</odometryFrame>

Commit message: fix the problem that subscriber "RLMemoryStore" can't run.

File: src/mp500lwa4d_description/urdf/base/base.gazebo.xacro (robot description, xacro)
@@ -16,5 +16,5 @@
           <kp>1000000.0</kp>
           <kd>100.0</kd>
-          <fdir1>0 0 1</fdir1>
+          <fdir1>0 0 2</fdir1>
           <material value="Gazebo/Grey"/>
       </gazebo>
@@ -26,5 +26,5 @@
           <kp>1000000.0</kp>
           <kd>100.0</kd>
-          <fdir1>0 0 1</fdir1>
+          <fdir1>0 0 2</fdir1>
           <material value="Gazebo/Grey"/>
       </gazebo>
@@ -32,9 +32,9 @@
       <gazebo reference="hanger">
           <gravity>true</gravity>
-          <mu1>0.1</mu1>
-          <mu2>0.1</mu2>
+          <mu1>100.5</mu1>
+          <mu2>100.5</mu2>
           <kp>1000000.0</kp>
           <kd>100.0</kd>
-          <fdir1>0 0 1</fdir1>
+          <fdir1>0 0 2</fdir1>
           <material value="Gazebo/Grey"/>
       </gazebo>

File: src/mp500lwa4d_description/urdf/base/base_mp500.urdf.xacro (robot description, xacro)
@@ -18,5 +18,5 @@
 	<link name="base_link">
 		<inertial>
-			<mass value="1" />
+			<mass value="100" />
 			<!--<origin xyz="0 0 0.216" rpy="0 0 0"/>-->
 			<!--<inertia ixx="0.54" ixy="0.0" ixz="0.0" iyy="1.08" iyz="0.0" izz="1.23" />-->
@@ -47,5 +47,5 @@
 	<link name="wheel_left_link" type="wheel">
 		<inertial>
-			<mass value="5" />
+			<mass value="1" />
 			<origin xyz="0 0 0" rpy="0 0 0" />
 			<inertia ixx="0.0045" ixy="0" ixz="0" iyy="0.0078" iyz="0" izz="0.0045" />
@@ -105,5 +105,5 @@
 	<link name="wheel_right_link" type="wheel">
 		<inertial>
-			<mass value="5" />
+			<mass value="1" />
 			<origin xyz="0 0 0" rpy="0 0 0" />
 			<!--inertia ixx="0.0051" ixy="0" ixz="0" iyy="0.0051" iyz="0" izz="0.009" /-->
@@ -136,5 +136,5 @@
 	<link name="hanger">
 		<inertial>
-			<mass value="5" />
+			<mass value="1" />
 			<origin xyz="0 0 0" rpy="0 0 0" />
 			<inertia ixx="0.0013" ixy="0" ixz="0" iyy="0.0013" iyz="0" izz="0.0013" />

Commit message: Organized files

File: src/mp500lwa4d_description/urdf/base/base.gazebo.xacro (robot description, xacro)
@@ -16,5 +16,5 @@
           <kp>1000000.0</kp>
           <kd>100.0</kd>
-          <fdir1>0 0 2</fdir1>
+          <fdir1>0 0 1</fdir1>
           <material value="Gazebo/Grey"/>
       </gazebo>
@@ -26,5 +26,5 @@
           <kp>1000000.0</kp>
           <kd>100.0</kd>
-          <fdir1>0 0 2</fdir1>
+          <fdir1>0 0 1</fdir1>
           <material value="Gazebo/Grey"/>
       </gazebo>
@@ -36,5 +36,5 @@
           <kp>1000000.0</kp>
           <kd>100.0</kd>
-          <fdir1>0 0 2</fdir1>
+          <fdir1>0 0 1</fdir1>
           <material value="Gazebo/Grey"/>
       </gazebo>

File: src/mp500lwa4d_description/urdf/base/base_mp500.urdf.xacro (robot description, xacro)
@@ -18,5 +18,5 @@
 	<link name="base_link">
 		<inertial>
-			<mass value="100" />
+			<mass value="10" />
 			<!--<origin xyz="0 0 0.216" rpy="0 0 0"/>-->
 			<!--<inertia ixx="0.54" ixy="0.0" ixz="0.0" iyy="1.08" iyz="0.0" izz="1.23" />-->
